Commit message: Added inertias to URDF file

File: puzzlebot_challenge/urdf/puzzlebot.urdf (robot description, URDF)
Before this commit: robot PuzzleBot, 5 links, 4 joints
Links:
- removed link base_footprint
- removed link wheel_coupler
- removed link wheel_coupler_2
- added link left_wheel, mass 0.0471238898038469; collision mesh filename=package://puzzlebot_challenge/models/MCR2_1000_1_1_Wheel_Co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; visual mesh filename=package://puzzlebot_challenge/models/MCR2_1000_1_1_Wheel_Co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
- added link right_wheel, mass 0.0471238898038469; collision mesh filename=package://puzzlebot_challenge/models/MCR2_1000_1_1_Wheel_Co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; visual mesh filename=package://puzzlebot_challenge/models/MCR2_1000_1_1_Wheel_Co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
- link base_link: mass None -> 0.0001; geometry 
- link chassis: mass None -> 0.9
Joints:
- removed joint base_footprint_joint
- joint wheel_coupler_joint: child wheel_coupler -> left_wheel; origin xyz=0 0 0 rpy=0 0 0 -> xyz=0.05 0.085 0.05 rpy=0 0 0
- joint wheel_coupler_joint_2: child wheel_coupler_2 -> right_wheel; origin xyz=0 0 0 rpy=0 0 0 -> xyz=0.05 -0.085 0.05 rpy=0 0 0

Commit message: Created puzzlebot_gazebo pkg and included lidar

File: puzzlebot_challenge/urdf/puzzlebot.urdf (robot description, URDF)
Before this commit: robot puzzlebot, 4 links, 3 joints
Links:
- added link rplidar_link; visual cylinder length=0.027 radius=0.035
Joints:
- removed joint wheel_coupler_joint
- removed joint wheel_coupler_joint_2
- added joint rplidar_joint: type fixed, parent chassis, child rplidar_link, origin xyz=0.05 0 0.16 rpy=0 0 0
- added joint wheel_left_joint: type continuous, parent chassis, child left_wheel, origin xyz=0.05 0.085 0.05 rpy=0 0 0, axis 0 1 0
- added joint wheel_right_joint: type continuous, parent chassis, child right_wheel, origin xyz=0.05 -0.085 0.05 rpy=0 0 0, axis 0 1 0

Commit message: Added sensors to Ignition

File: puzzlebot_challenge/urdf/puzzlebot.urdf (robot description, URDF)
Before this commit: robot puzzlebot, 5 links, 4 joints
Links:
- added link camera_link, mass 0.01; visual box size=0.04 0.02 0.02
- link rplidar_link: mass None -> 0.1
Joints:
- added joint camera_joint: type fixed, parent chassis, child camera_link, origin xyz=0.1 0 0.1 rpy=0 0 0

Commit message: vision temporal fix, usable in sim

File: puzzlebot_challenge/urdf/puzzlebot.urdf (robot description, URDF)
Before this commit: robot puzzlebot, 6 links, 5 joints
Links:
- link camera_link: geometry visual box size=0.02 0.02 0.02
Joints:
- joint camera_joint: origin xyz=0.1 0 0.1 rpy=0 0 0 -> xyz=0.1 0 0.08 rpy=0 0 0
- joint rplidar_joint: origin xyz=0.05 0 0.16 rpy=0 0 0 -> xyz=0.05 0 0.16 rpy=0 3.14 0
- joint wheel_left_joint: origin xyz=0.05 0.085 0.05 rpy=0 0 0 -> xyz=0.05 0.09 0.05 rpy=0 0 0
- joint wheel_right_joint: origin xyz=0.05 -0.085 0.05 rpy=0 0 0 -> xyz=0.05 -0.09 0.05 rpy=0 0 0

Commit message: added more arucos, removed handler for lifter

File: puzzlebot_challenge/urdf/puzzlebot.urdf (robot description, URDF)
Before this commit: robot puzzlebot, 6 links, 5 joints
Links:
- link chassis: mass 0.9 -> 0.8
- link left_wheel: mass 0.0471238898038469 -> 0.05
- link right_wheel: mass 0.0471238898038469 -> 0.05
Joints:
- joint wheel_left_joint: limit (none) -> lower=-1.79769e+308 upper=1.79769e+308 effort=1 velocity=6; type continuous -> revolute
- joint wheel_right_joint: limit (none) -> lower=-1.79769e+308 upper=1.79769e+308 effort=1 velocity=6; type continuous -> revolute

Commit message: Adjusted lidar frame to match the real data

File: puzzlebot_challenge/urdf/puzzlebot.urdf (robot description, URDF)
Before this commit: robot puzzlebot, 6 links, 5 joints
Joints:
- joint rplidar_joint: origin xyz=0.05 0 0.16 rpy=0 3.14 0 -> xyz=0.05 0 0.16 rpy=3.1416 3.14 0

Commit message: Changed camera topic, change the launch file that runs the aruco node

File: puzzlebot_challenge/urdf/puzzlebot.urdf (robot description, URDF)
Before this commit: robot puzzlebot, 6 links, 5 joints
Joints:
- joint rplidar_joint: origin xyz=0.05 0 0.16 rpy=3.1416 3.14 0 -> xyz=0.05 0 0.16 rpy=3.1416 3.1416 0
